Commit message: Todo: how to link btw dynamixel input and mvgroup?

File: franka_panda_description/robots/hand_withcam.xacro (robot description, xacro)
@@ -22,61 +22,8 @@
       <inertial>
         <origin rpy="0 0 0" xyz="0 0.0015244 -0.0275912"/>
-        <mass value="0.73"/>
+        <mass value="0.704"/>
         <inertia ixx="0.00278560230025" ixy="0.0" ixz="0.0" iyy="0.000400033405336" iyz="0.0" izz="0.00256378041832"/>
       </inertial>
     </link>
-    <link name="${ns}_leftfinger">
-      <visual>
-        <geometry>
-          <mesh filename="package://franka_panda_description/meshes/visual/finger.dae"/>
-        </geometry>
-      </visual>
-      <collision>
-        <geometry>
-          <mesh filename="package://franka_panda_description/meshes/collision/finger.stl"/>
-        </geometry>
-      </collision>
-      <inertial>
-        <origin rpy="0 0 0" xyz="0 0.0145644 -0.0027941"/>
-        <mass value="0.1"/>
-        <inertia ixx="3.01220925051e-05" ixy="0.0" ixz="0.0" iyy="2.95873808038e-05" iyz="0.0" izz="6.95125211657e-06"/>
-      </inertial>
-    </link>
-    <link name="${ns}_rightfinger">
-      <visual>
-        <origin xyz="0 0 0" rpy="0 0 ${pi}"/>
-        <geometry>
-          <mesh filename="package://franka_panda_description/meshes/visual/finger.dae"/>
-        </geometry>
-      </visual>
-      <collision>
-        <origin xyz="0 0 0" rpy="0 0 ${pi}"/>
-        <geometry>
-          <mesh filename="package://franka_panda_description/meshes/collision/finger.stl"/>
-        </geometry>
-      </collision>
-      <inertial>
-        <origin rpy="0 0 3.141592653589793" xyz="0 -0.0145644 0.0027941"/>
-        <mass value="0.1"/>
-        <inertia ixx="3.01220925051e-05" ixy="0.0" ixz="0.0" iyy="2.95873808038e-05" iyz="0.0" izz="6.95125211657e-06"/>
-      </inertial>
-    </link>
-    <joint name="${ns}_finger_joint1" type="prismatic">
-      <parent link="${ns}_hand"/>
-      <child link="${ns}_leftfinger"/>
-      <origin xyz="0 0 0.0084" rpy="0 0 0"/>
-      <axis xyz="0 1 0"/>
-      <limit effort="20" lower="0.0" upper="0.04" velocity="0.2"/>
-      <dynamics damping="500.0" friction="0.0"/>
-    </joint>
-    <joint name="${ns}_finger_joint2" type="prismatic">
-      <parent link="${ns}_hand"/>
-      <child link="${ns}_rightfinger"/>
-      <origin xyz="0 0 0.0084" rpy="0 0 0"/>
-      <axis xyz="0 -1 0"/>
-      <limit effort="20" lower="0.0" upper="0.04" velocity="0.2"/>
-      <dynamics damping="500.0" friction="0.0"/>
-      <mimic joint="${ns}_finger_joint1" />
-    </joint>
   </xacro:macro>
 </robot>

File: franka_panda_description/robots/panda_arm_hand.urdf.xacro (robot description, xacro)
@@ -8,5 +8,5 @@
   <xacro:include filename="$(find franka_panda_description)/robots/panda_arm.xacro"/>
   <xacro:if value="$(arg load_gripper)">
-    <xacro:include filename="$(find franka_panda_description)/robots/hand_withcam.xacro"/>
+    <xacro:include filename="$(find franka_panda_description)/robots/hand.xacro"/>
     <xacro:hand ns="panda" rpy="0 0 ${-pi/4}" connected_to="panda_link8"/>
   </xacro:if>

File: franka_panda_description/robots/panda_arm_hand_screwsort.urdf.xacro (robot description, xacro)
@@ -8,5 +8,5 @@
   <xacro:include filename="$(find franka_panda_description)/robots/panda_arm.xacro"/>
   <xacro:if value="$(arg load_gripper)">
-    <xacro:include filename="$(find franka_panda_description)/robots/hand_withcam.xacro"/>
+    <xacro:include filename="$(find franka_panda_description)/robots/hand_screwgripper.xacro"/>
     <xacro:hand ns="panda" rpy="0 0 ${-pi/4}" connected_to="panda_link8"/>
   </xacro:if>
